Commit message: Update arm_assy_backup.xacro

File: URDF/arm_assy_backup_description/urdf/arm_assy_backup.xacro (robot description, xacro)
@@ -26,7 +26,7 @@
 <link name="armA_1">
   <inertial>
-    <origin rpy="0 0 0" xyz="0.013334027173307894 0.01626500178908685 0.016722436439834704"/>
-    <mass value="0.37431007884671536"/>
-    <inertia ixx="0.001123" ixy="-0.000406" ixz="-0.000201" iyy="0.00095" iyz="-0.000246" izz="0.001166"/>
+    <origin rpy="0 0 0" xyz="0.016036 0.000156 0.01673"/>
+    <mass value="0.647"/>
+    <inertia ixx="0.0010747" ixy="-0.00001386" ixz="-0.00045398" iyy="0.002177" iyz="-0.000005806" izz="0.0018872"/>
   </inertial>
   <visual>
@@ -46,7 +46,7 @@
 <link name="armB_1">
   <inertial>
-    <origin rpy="0 0 0" xyz="0.03355630303953762 -0.062499232501169635 -0.022605136354354627"/>
-    <mass value="0.18361177429179534"/>
-    <inertia ixx="0.000375" ixy="0.000138" ixz="4e-06" iyy="0.00011" iyz="-7e-06" izz="0.000429"/>
+    <origin rpy="0 0 0" xyz="0.095476 0.004053 -0.028703"/>
+    <mass value="0.273"/>
+    <inertia ixx="0.000592" ixy="0.000034987" ixz="0.000383933" iyy="0.001323383" iyz="-0.000038358" izz="0.000831039"/>
   </inertial>
   <visual>
